Commit message: clover_description: Tweak parameters a bit, add collision boxes

File: clover_description/urdf/drones/clover4_physics.xacro (robot description, xacro)
@@ -9,6 +9,6 @@
   <xacro:property name="mesh_scale_prop" value="0.001 0.001 0.001"/>
   <xacro:property name="mass" value="0.5" /> <!-- [kg] -->
-  <xacro:property name="body_width" value="0.47" /> <!-- [m] -->
-  <xacro:property name="body_height" value="0.11" /> <!-- [m] -->
+  <xacro:property name="body_width" value="0.35" /> <!-- [m] -->
+  <xacro:property name="body_height" value="0.124" /> <!-- [m] -->
   <xacro:property name="mass_rotor" value="0.01" /> <!-- [kg] -->
   <xacro:property name="arm_length_front_x" value="0.083" /> <!-- [m] -->
@@ -17,5 +17,5 @@
   <xacro:property name="arm_length_back_y" value="0.083" /> <!-- [m] -->
   <xacro:property name="rotor_offset_top" value="0.023" /> <!-- [m] -->
-  <xacro:property name="radius_rotor" value="0.128" /> <!-- [m] -->
+  <xacro:property name="radius_rotor" value="0.06" /> <!-- [m] -->
   <xacro:property name="motor_constant" value="8.54858e-06" /> <!-- [kg.m/s^2] -->
   <xacro:property name="moment_constant" value="0.06" /> <!-- [m] -->

File: clover_description/urdf/drones/clover_base.xacro (robot description, xacro)
@@ -22,5 +22,5 @@
   <xacro:arg name='use_tcp' default='true' />
   <xacro:arg name='vehicle_is_tailsitter' default='false' />
-  <xacro:arg name='visual_material' default='DarkGrey' />
+  <xacro:arg name='visual_material' default='Grey' />
   <xacro:arg name='enable_mavlink_interface' default='true' />
   <xacro:arg name='enable_wind' default='false' />

File: clover_description/urdf/multirotor_base.xacro (robot description, xacro)
@@ -33,5 +33,6 @@
       </inertial>
       <visual>
-        <origin xyz="0 0 0" rpy="0 0 0" />
+        <!-- Shift the mesh down, since its origin is not at center -->
+        <origin xyz="0 0 ${-body_height/2}" rpy="0 0 0" />
         <geometry>
           <mesh filename="package://clover_description/meshes/${mesh_file}"
@@ -40,8 +41,34 @@
         </geometry>
       </visual>
-      <collision>
-        <origin xyz="0 0 0" rpy="0 0 0" />
+      <!-- FIXME: Add proper collision boxes -->
+      <!-- FIXME: Maybe add these boxes in a separate macro? -->
+      <collision name="body_collision_box">
+        <origin xyz="0 0 ${body_height/4}" rpy="0 0 0" />
         <geometry>
-          <box size="${body_width} ${body_width} ${body_height}" /> <!-- [m] [m] [m] -->
+          <box size="${body_width} ${body_width} ${body_height/2}" /> <!-- [m] [m] [m] -->
+        </geometry>
+      </collision>
+      <collision name="front_left_leg_collision_box">
+        <origin xyz="${-body_width/5} ${body_width/5} ${-body_height/4}" rpy="0 0 0" />
+        <geometry>
+          <box size="${body_width/15} ${body_width/15} ${body_height/2}" /> <!-- [m] [m] [m] -->
+        </geometry>
+      </collision>
+      <collision name="front_right_leg_collision_box">
+        <origin xyz="${body_width/5} ${body_width/5} ${-body_height/4}" rpy="0 0 0" />
+        <geometry>
+          <box size="${body_width/15} ${body_width/15} ${body_height/2}" /> <!-- [m] [m] [m] -->
+        </geometry>
+      </collision>
+      <collision name="back_left_leg_collision_box">
+        <origin xyz="${-body_width/5} ${-body_width/5} ${-body_height/4}" rpy="0 0 0" />
+        <geometry>
+          <box size="${body_width/15} ${body_width/15} ${body_height/2}" /> <!-- [m] [m] [m] -->
+        </geometry>
+      </collision>
+      <collision name="back_right_leg_collision_box">
+        <origin xyz="${body_width/5} ${-body_width/5} ${-body_height/4}" rpy="0 0 0" />
+        <geometry>
+          <box size="${body_width/15} ${body_width/15} ${body_height/2}" /> <!-- [m] [m] [m] -->
         </geometry>
       </collision>
