Commit message: clover_description: Add option to use throttling_camera

File: clover_description/urdf/camera_sensor.urdf.xacro (robot description, xacro)
@@ -2,5 +2,5 @@
 <robot name="camera_sensor" xmlns:xacro="http://ros.org/wiki/xacro">
   <xacro:macro name="camera_sensor_base"
-      params="name width height rate horizontal_fov frame_name k1 k2 k3 p1 p2 cx cy cx_prime">
+      params="name width height rate horizontal_fov frame_name k1 k2 k3 p1 p2 cx cy cx_prime ros_plugin_name min_rate window_size max_st_dev">
     <gazebo reference="${name}_link">
       <sensor type="camera" name="${name}">
@@ -28,5 +28,5 @@
         <update_rate>${rate}</update_rate>
         <visualize>1</visualize>
-        <plugin name="camera_plugin" filename="libgazebo_ros_camera.so">
+        <plugin name="camera_plugin" filename="${ros_plugin_name}">
           <alwaysOn>true</alwaysOn>
           <imageTopicName>image_raw</imageTopicName>
@@ -43,9 +43,19 @@
           <distortionT1>${p1}</distortionT1>
           <distortionT2>${p2}</distortionT2>
+          <!-- throttling_camera specific options start here -->
+          <minUpdateRate>${min_rate}</minUpdateRate>
+          <windowSize>${window_size}</windowSize>
+          <maxStDev>${max_st_dev}</maxStDev>
         </plugin>
       </sensor>
     </gazebo>
   </xacro:macro>
-  <xacro:macro name="camera_sensor" params="name width height rate horizontal_fov k1:=0 k2:=0 k3:=0 p1:=0 p2:=0">
+  <xacro:macro name="camera_sensor" params="name width height rate horizontal_fov k1:=0 k2:=0 k3:=0 p1:=0 p2:=0 do_throttling:=false">
+    <xacro:if value="${do_throttling}">
+      <xacro:property name="ros_plugin_name" value="libthrottling_camera.so"/>
+    </xacro:if>
+    <xacro:unless value="${do_throttling}">
+      <xacro:property name="ros_plugin_name" value="libgazebo_ros_camera.so"/>
+    </xacro:unless>
     <xacro:camera_sensor_base
       name="${name}"
@@ -63,4 +73,8 @@
       cy="${(height + 1.0)/2.0}"
       cx_prime="${(width + 1.0)/2.0}"
+      ros_plugin_name="${ros_plugin_name}"
+      min_rate="${rate * 0.95}"
+      window_size="${rate}"
+      max_st_dev="${3.0 / rate}"
     />
   </xacro:macro>

File: clover_description/urdf/clover/clover4.xacro (robot description, xacro)
@@ -5,4 +5,5 @@
   <xacro:arg name="led" default="true"/>
   <xacro:arg name="gps" default="true"/>
+  <xacro:arg name="maintain_camera_rate" default="false"/>
   <xacro:include filename="$(find clover_description)/urdf/clover/clover4_base.xacro" />
   <xacro:include filename="$(find clover_description)/urdf/sensors/rpi_cam.urdf.xacro"/>
@@ -11,5 +12,5 @@
   <!-- Create camera plugin -->
   <xacro:if value="$(arg main_camera)">
-    <xacro:rpi_cam name="main_camera" parent="base_link" x="0.055" y="0.0" z="-0.03" roll="0" pitch="${pi / 2}" yaw="0" width="320" height="240" rate="40"/>
+    <xacro:rpi_cam name="main_camera" parent="base_link" x="0.055" y="0.0" z="-0.03" roll="0" pitch="${pi / 2}" yaw="0" width="320" height="240" rate="40" do_throttling="$(arg maintain_camera_rate)"/>
   </xacro:if>
   <!-- Create rangefinder plugin -->

File: clover_description/urdf/sensors/rpi_cam.urdf.xacro (robot description, xacro)
@@ -2,5 +2,5 @@
 <robot name="rpi_camera" xmlns:xacro="http://ros.org/wiki/xacro">
   <xacro:include filename="$(find clover_description)/urdf/camera_sensor.urdf.xacro"/>
-  <xacro:macro name="rpi_cam" params="name:=rpi_cam parent x:=0 y:=0 z:=0 roll:=0 pitch:=0 yaw:=0 width:=320 height:=240 rate:=40">
+  <xacro:macro name="rpi_cam" params="name:=rpi_cam parent x:=0 y:=0 z:=0 roll:=0 pitch:=0 yaw:=0 width:=320 height:=240 rate:=40 do_throttling:=false">
     <joint name="${name}_joint" type="fixed">
       <origin xyz="${x} ${y} ${z}"
@@ -52,4 +52,5 @@
       rate="${rate}"
       horizontal_fov="${120 * pi / 180}"
+      do_throttling="${do_throttling}"
     />
   </xacro:macro>
