Commit message: clover_description: Prevent lumping for camera link/joint

File: clover_description/urdf/sensors/rpi_cam.urdf.xacro (robot description, xacro)
@@ -3,8 +3,8 @@
   <xacro:include filename="$(find clover_description)/urdf/constants.urdf.xacro"/>
   <xacro:include filename="$(find clover_description)/urdf/camera_sensor.urdf.xacro"/>
-  <xacro:macro name="rpi_cam" params="name:=rpi_cam parent x:=0 y:=0 z:=0 r:=0 p:=0 y:=0">
+  <xacro:macro name="rpi_cam" params="name:=rpi_cam parent x:=0 y:=0 z:=0 roll:=0 pitch:=0 yaw:=0">
     <joint name="${name}_joint" type="fixed">
       <origin xyz="${x} ${y} ${z}"
-              rpy="${r} ${p} ${y}"/>
+              rpy="${roll} ${pitch} ${yaw}"/>
       <parent link="${parent}"/>
       <child link="${name}_link"/>
@@ -29,6 +29,10 @@
       </inertial>
     </link>
+    <gazebo reference="${name}_joint">
+      <disableFixedJointLumping>true</disableFixedJointLumping>
+      <preserveFixedJoint>true</preserveFixedJoint>
+    </gazebo>
     <camera_sensor name="${name}" width="320" height="240" rate="40" horizontal_fov="${120*M_PI/180}"/>
   </xacro:macro>
-  <rpi_cam name="main_camera" parent="drone"/>
+  <!-- <rpi_cam name="main_camera" parent="base_link"/> -->
 </robot>

Commit message: clover_description: Allow setting width/height for rpi_cam

File: clover_description/urdf/sensors/rpi_cam.urdf.xacro (robot description, xacro)
@@ -3,5 +3,5 @@
   <xacro:include filename="$(find clover_description)/urdf/constants.urdf.xacro"/>
   <xacro:include filename="$(find clover_description)/urdf/camera_sensor.urdf.xacro"/>
-  <xacro:macro name="rpi_cam" params="name:=rpi_cam parent x:=0 y:=0 z:=0 roll:=0 pitch:=0 yaw:=0">
+  <xacro:macro name="rpi_cam" params="name:=rpi_cam parent x:=0 y:=0 z:=0 roll:=0 pitch:=0 yaw:=0 width:=320 height:=240 rate:=40">
     <joint name="${name}_joint" type="fixed">
       <origin xyz="${x} ${y} ${z}"
@@ -14,5 +14,5 @@
         <origin xyz="0 0 0" rpy="0 0 0"/>
         <geometry>
-          <box size="0.01 0.01 0.01"/>
+          <box size="0.005 0.005 0.005"/>
         </geometry>
       </visual>
@@ -20,5 +20,5 @@
         <origin xyz="0 0 0" rpy="0 0 0"/>
         <geometry>
-          <box size="0.01 0.01 0.01"/>
+          <box size="0.005 0.005 0.005"/>
         </geometry>
       </collision>
@@ -33,5 +33,5 @@
       <preserveFixedJoint>true</preserveFixedJoint>
     </gazebo>
-    <camera_sensor name="${name}" width="320" height="240" rate="40" horizontal_fov="${120*M_PI/180}"/>
+    <camera_sensor name="${name}" width="${width}" height="${height}" rate="${rate}" horizontal_fov="${120*M_PI/180}"/>
   </xacro:macro>
   <!-- <rpi_cam name="main_camera" parent="base_link"/> -->
