Commit message: clover_description: Add leg colliders

File: clover_description/urdf/clover/clover4_macros.xacro (robot description, xacro)
@@ -62,8 +62,32 @@
            - sfalexrog
       -->
-      <collision>
-        <origin xyz="0 0 0" rpy="0 0 0" />
-        <geometry>
-          <box size="${body_width} ${body_width} ${body_height}" /> <!-- [m] [m] [m] -->
+      <collision name="upper_body">
+        <origin xyz="0 0 ${body_height/4}" rpy="0 0 0" />
+        <geometry>
+          <box size="${body_width} ${body_width} ${body_height/2}" /> <!-- [m] [m] [m] -->
+        </geometry>
+      </collision>
+      <collision name="front_left_leg">
+        <origin xyz="${body_width/5} ${body_width/5} ${-body_height/4}" rpy="0 0 0" />
+        <geometry>
+          <box size="${body_width/10} ${body_width/10} ${body_height/2}" /> <!-- [m] [m] [m] -->
+        </geometry>
+      </collision>
+      <collision name="front_right_leg">
+        <origin xyz="${body_width/5} ${-body_width/5} ${-body_height/4}" rpy="0 0 0" />
+        <geometry>
+          <box size="${body_width/10} ${body_width/10} ${body_height/2}" /> <!-- [m] [m] [m] -->
+        </geometry>
+      </collision>
+      <collision name="back_left_leg">
+        <origin xyz="${-body_width/5} ${body_width/5} ${-body_height/4}" rpy="0 0 0" />
+        <geometry>
+          <box size="${body_width/10} ${body_width/10} ${body_height/2}" /> <!-- [m] [m] [m] -->
+        </geometry>
+      </collision>
+      <collision name="back_right_leg">
+        <origin xyz="${-body_width/5} ${-body_width/5} ${-body_height/4}" rpy="0 0 0" />
+        <geometry>
+          <box size="${body_width/10} ${body_width/10} ${body_height/2}" /> <!-- [m] [m] [m] -->
         </geometry>
       </collision>

Commit message: clover_description: Revert adding additional colliders
Unfortunately, this breaks physics too much

File: clover_description/urdf/clover/clover4_macros.xacro (robot description, xacro)
@@ -62,26 +62,8 @@
            - sfalexrog
       -->
-      <collision name="upper_body">
-        <origin xyz="0 0 ${body_height/4}" rpy="0 0 0" />
-        <geometry>
-          <box size="${body_width} ${body_width} ${body_height/2}" /> <!-- [m] [m] [m] -->
-        </geometry>
-      </collision>
-      <collision name="front_left_leg">
-        <origin xyz="${body_width/5} ${body_width/5} ${-body_height/4}" rpy="0 0 0" />
-        <geometry>
-          <box size="${body_width/10} ${body_width/10} ${body_height/2}" /> <!-- [m] [m] [m] -->
-        </geometry>
-      </collision>
-      <collision name="front_right_leg">
-        <origin xyz="${body_width/5} ${-body_width/5} ${-body_height/4}" rpy="0 0 0" />
-        <geometry>
-          <box size="${body_width/10} ${body_width/10} ${body_height/2}" /> <!-- [m] [m] [m] -->
-        </geometry>
-      </collision>
-      <collision name="back_left_leg">
-        <origin xyz="${-body_width/5} ${body_width/5} ${-body_height/4}" rpy="0 0 0" />
-        <geometry>
-          <box size="${body_width/10} ${body_width/10} ${body_height/2}" /> <!-- [m] [m] [m] -->
+      <collision>
+        <origin xyz="0 0 0" rpy="0 0 0" />
+        <geometry>
+          <box size="${body_width} ${body_width} ${body_height}" /> <!-- [m] [m] [m] -->
         </geometry>
       </collision>

Commit message: clover_description: Tweak drone physics, make it more bouncy

File: clover_description/urdf/clover/clover4_macros.xacro (robot description, xacro)
@@ -68,10 +68,4 @@
         </geometry>
       </collision>
-      <collision name="back_right_leg">
-        <origin xyz="${-body_width/5} ${-body_width/5} ${-body_height/4}" rpy="0 0 0" />
-        <geometry>
-          <box size="${body_width/10} ${body_width/10} ${body_height/2}" /> <!-- [m] [m] [m] -->
-        </geometry>
-      </collision>
     </link>
     <!-- This link is here for a single reason: to draw transparent parts (oh, and also to be the bane of my existence).
@@ -156,17 +150,8 @@
     </gazebo>
     <gazebo reference="base_link">
-      <collision name='base_link_inertia_collision'>
-        <surface>
-          <contact>
-            <ode>
-              <min_depth>0.001</min_depth>
-              <max_vel>0.0</max_vel>
-            </ode>
-          </contact>
-          <friction>
-            <ode/>
-          </friction>
-        </surface>
-      </collision>
+      <kp>10000.0</kp>
+      <kd>10.0</kd>
+      <maxVel>10.0</maxVel>
+      <minDepth>0.001</minDepth>
    </gazebo>
   </xacro:macro>
