Commit message: clover_description: Set rangefinder min range outside drone collider

File: clover_description/urdf/clover/clover4_camera.xacro (robot description, xacro)
@@ -5,4 +5,4 @@
   <xacro:include filename="$(find clover_description)/urdf/sensors/distance_sensor.urdf.xacro"/>
   <xacro:rpi_cam name="main_camera" parent="base_link" x="0.055" y="0.0" z="-0.03" roll="0" pitch="${M_PI / 2}" yaw="0" width="320" height="240" rate="40"/>
-  <xacro:distance_sensor parent="base_link" x="0.0" y="0.0" z="-0.03" roll="0" pitch="${M_PI / 2}" yaw="0"/>
+  <xacro:distance_sensor parent="base_link" x="0.0" y="0.0" z="-0.04" roll="0" pitch="${M_PI / 2}" yaw="0"/>
 </robot>

File: clover_description/urdf/sensors/distance_sensor.urdf.xacro (robot description, xacro)
@@ -14,5 +14,5 @@
         <origin xyz="0 0 0" rpy="0 0 0"/>
         <geometry>
-          <box size="0.005 0.005 0.001"/>
+          <box size="0.001 0.005 0.005"/>
         </geometry>
       </visual>
@@ -20,5 +20,5 @@
         <origin xyz="0 0 0" rpy="0 0 0"/>
         <geometry>
-          <box size="0.001 0.005 0.005"/>
+          <box size="0.001 0.001 0.005"/>
         </geometry>
       </collision>
@@ -46,5 +46,5 @@
           </scan>
           <range>
-            <min>${range_min}</min>
+            <min>0.03</min> <!-- Note: This is a hack, since the rangefinder is inside the drone collision box -->
             <max>${range_max}</max>
             <resolution>${resolution}</resolution>
