Commit message: Add hardcoded URDF LED strip

File: clover_description/urdf/clover/clover4.xacro (robot description, xacro)
@@ -3,4 +3,5 @@
   <xacro:arg name="main_camera" default="true"/>
   <xacro:arg name="rangefinder" default="true"/>
+  <xacro:arg name="led" default="true"/>
   <xacro:arg name="gps" default="true"/>
   <xacro:include filename="$(find clover_description)/urdf/clover/clover4_base.xacro" />
@@ -15,4 +16,254 @@
     <xacro:distance_sensor parent="base_link" x="0.0" y="0.0" z="-0.04" roll="0" pitch="${M_PI / 2}" yaw="0"/>
   </xacro:if>
+  <!-- Add LED strip model TODO: redo -->
+  <joint name="led_strip_joint" type="fixed">
+    <origin xyz="0 0 0"
+            rpy="0 0 0"/>
+    <parent link="base_link"/>
+    <child link="led_link"/>
+  </joint>
+  <!-- TODO: remove hardcode -->
+  <link name="led_link">
+    <visual name="led_0_visual">
+      <origin rpy="0  0  0" xyz="0    0.08  0"/>
+      <geometry>
+        <sphere radius="0.005"/>
+      </geometry>
+    </visual>
+    <visual name="led_1_visual">
+      <origin rpy="0  0  0" xyz="0.01251  0.07901  0"/>
+      <geometry>
+        <sphere radius="0.005"/>
+      </geometry>
+    </visual>
+    <visual name="led_2_visual">
+      <origin rpy="0  0  0" xyz="0.02472  0.07608  0"/>
+      <geometry>
+        <sphere radius="0.005"/>
+      </geometry>
+    </visual>
+    <visual name="led_3_visual">
+      <origin rpy="0  0  0" xyz="0.03631  0.07128  0"/>
+      <geometry>
+        <sphere radius="0.005"/>
+      </geometry>
+    </visual>
+    <visual name="led_4_visual">
+      <origin rpy="0  0  0" xyz="0.04702  0.06472  0"/>
+      <geometry>
+        <sphere radius="0.005"/>
+      </geometry>
+    </visual>
+    <visual name="led_5_visual">
+      <origin rpy="0  0  0" xyz="0.05656  0.05656  0"/>
+      <geometry>
+        <sphere radius="0.005"/>
+      </geometry>
+    </visual>
+    <visual name="led_6_visual">
+      <origin rpy="0  0  0" xyz="0.06472  0.04702  0"/>
+      <geometry>
+        <sphere radius="0.005"/>
+      </geometry>
+    </visual>
+    <visual name="led_7_visual">
+      <origin rpy="0  0  0" xyz="0.07128  0.03631  0"/>
+      <geometry>
+        <sphere radius="0.005"/>
+      </geometry>
+    </visual>
+    <visual name="led_8_visual">
+      <origin rpy="0  0  0" xyz="0.07608  0.02472  0"/>
+      <geometry>
+        <sphere radius="0.005"/>
+      </geometry>
+    </visual>
+    <visual name="led_9_visual">
+      <origin rpy="0  0  0" xyz="0.07901  0.01251  0"/>
+      <geometry>
+        <sphere radius="0.005"/>
+      </geometry>
+    </visual>
+    <visual name="led_10_visual">
+      <origin rpy="0  0  0" xyz="0.08  0    0"/>
+      <geometry>
+        <sphere radius="0.005"/>
+      </geometry>
+    </visual>
+    <visual name="led_11_visual">
+      <origin rpy="0  0  0" xyz="0.07901 -0.01251  0"/>
+      <geometry>
+        <sphere radius="0.005"/>
+      </geometry>
+    </visual>
+    <visual name="led_12_visual">
+      <origin rpy="0  0  0" xyz="0.07608 -0.02472  0"/>
+      <geometry>
+        <sphere radius="0.005"/>
+      </geometry>
+    </visual>
+    <visual name="led_13_visual">
+      <origin rpy="0  0  0" xyz="0.07128 -0.03631  0"/>
+      <geometry>
+        <sphere radius="0.005"/>
+      </geometry>
+    </visual>
+    <visual name="led_14_visual">
+      <origin rpy="0  0  0" xyz="0.06472 -0.04702  0"/>
+      <geometry>
+        <sphere radius="0.005"/>
+      </geometry>
+    </visual>
+    <visual name="led_15_visual">
+      <origin rpy="0  0  0" xyz="0.05656 -0.05656  0"/>
+      <geometry>
+        <sphere radius="0.005"/>
+      </geometry>
+    </visual>
+    <visual name="led_16_visual">
+      <origin rpy="0  0  0" xyz="0.04702 -0.06472  0"/>
+      <geometry>
+        <sphere radius="0.005"/>
+      </geometry>
+    </visual>
+    <visual name="led_17_visual">
+      <origin rpy="0  0  0" xyz="0.03631 -0.07128  0"/>
+      <geometry>
+        <sphere radius="0.005"/>
+      </geometry>
+    </visual>
+    <visual name="led_18_visual">
+      <origin rpy="0  0  0" xyz="0.02472 -0.07608  0"/>
+      <geometry>
+        <sphere radius="0.005"/>
+      </geometry>
+    </visual>
+    <visual name="led_19_visual">
+      <origin rpy="0  0  0" xyz="0.01251 -0.07901  0"/>
+      <geometry>
+        <sphere radius="0.005"/>
+      </geometry>
+    </visual>
+    <visual name="led_20_visual">
+      <origin rpy="0  0  0" xyz="0   -0.08  0"/>
+      <geometry>
+        <sphere radius="0.005"/>
+      </geometry>
+    </visual>
+    <visual name="led_21_visual">
+      <origin rpy="0  0  0" xyz="-0.01251 -0.07901  0"/>
+      <geometry>
+        <sphere radius="0.005"/>
+      </geometry>
+    </visual>
+    <visual name="led_22_visual">
+      <origin rpy="0  0  0" xyz="-0.02472 -0.07608  0"/>
+      <geometry>
+        <sphere radius="0.005"/>
+      </geometry>
+    </visual>
+    <visual name="led_23_visual">
+      <origin rpy="0  0  0" xyz="-0.03631 -0.07128  0"/>
+      <geometry>
+        <sphere radius="0.005"/>
+      </geometry>
+    </visual>
+    <visual name="led_24_visual">
+      <origin rpy="0  0  0" xyz="-0.04702 -0.06472  0"/>
+      <geometry>
+        <sphere radius="0.005"/>
+      </geometry>
+    </visual>
+    <visual name="led_25_visual">
+      <origin rpy="0  0  0" xyz="-0.05656 -0.05656  0"/>
+      <geometry>
+        <sphere radius="0.005"/>
+      </geometry>
+    </visual>
+    <visual name="led_26_visual">
+      <origin rpy="0  0  0" xyz="-0.06472 -0.04702  0"/>
+      <geometry>
+        <sphere radius="0.005"/>
+      </geometry>
+    </visual>
+    <visual name="led_27_visual">
+      <origin rpy="0  0  0" xyz="-0.07128 -0.03631  0"/>
+      <geometry>
+        <sphere radius="0.005"/>
+      </geometry>
+    </visual>
+    <visual name="led_28_visual">
+      <origin rpy="0  0  0" xyz="-0.07608 -0.02472  0"/>
+      <geometry>
+        <sphere radius="0.005"/>
+      </geometry>
+    </visual>
+    <visual name="led_29_visual">
+      <origin rpy="0  0  0" xyz="-0.07901 -0.01251  0"/>
+      <geometry>
+        <sphere radius="0.005"/>
+      </geometry>
+    </visual>
+    <visual name="led_30_visual">
+      <origin rpy="0  0  0" xyz="-0.08  0    0"/>
+      <geometry>
+        <sphere radius="0.005"/>
+      </geometry>
+    </visual>
+    <visual name="led_31_visual">
+      <origin rpy="0  0  0" xyz="-0.07901  0.01251  0"/>
+      <geometry>
+        <sphere radius="0.005"/>
+      </geometry>
+    </visual>
+    <visual name="led_32_visual">
+      <origin rpy="0  0  0" xyz="-0.07608  0.02472  0"/>
+      <geometry>
+        <sphere radius="0.005"/>
+      </geometry>
+    </visual>
+    <visual name="led_33_visual">
+      <origin rpy="0  0  0" xyz="-0.07128  0.03631  0"/>
+      <geometry>
+        <sphere radius="0.005"/>
+      </geometry>
+    </visual>
+    <visual name="led_34_visual">
+      <origin rpy="0  0  0" xyz="-0.06472  0.04702  0"/>
+      <geometry>
+        <sphere radius="0.005"/>
+      </geometry>
+    </visual>
+    <visual name="led_35_visual">
+      <origin rpy="0  0  0" xyz="-0.05656  0.05656  0"/>
+      <geometry>
+        <sphere radius="0.005"/>
+      </geometry>
+    </visual>
+    <visual name="led_36_visual">
+      <origin rpy="0  0  0" xyz="-0.04702  0.06472  0"/>
+      <geometry>
+        <sphere radius="0.005"/>
+      </geometry>
+    </visual>
+    <visual name="led_37_visual">
+      <origin rpy="0  0  0" xyz="-0.03631  0.07128  0"/>
+      <geometry>
+        <sphere radius="0.005"/>
+      </geometry>
+    </visual>
+    <visual name="led_38_visual">
+      <origin rpy="0  0  0" xyz="-0.02472  0.07608  0"/>
+      <geometry>
+        <sphere radius="0.005"/>
+      </geometry>
+    </visual>
+    <visual name="led_39_visual">
+      <origin rpy="0  0  0" xyz="-0.01251  0.07901  0"/>
+      <geometry>
+        <sphere radius="0.005"/>
+      </geometry>
+    </visual>
+  </link>
   <xacro:if value="$(arg gps)">
     <!-- Instantiate gps plugin. -->

Commit message: clover_description: Add LED xarco model
clover_simulation: Implement LED visual plugin and controller

File: clover_description/urdf/clover/clover4.xacro (robot description, xacro)
@@ -8,4 +8,5 @@
   <xacro:include filename="$(find clover_description)/urdf/sensors/rpi_cam.urdf.xacro"/>
   <xacro:include filename="$(find clover_description)/urdf/sensors/distance_sensor.urdf.xacro"/>
+  <xacro:include filename="$(find clover_description)/urdf/leds/led_strip.xacro"/>
   <!-- Create camera plugin -->
   <xacro:if value="$(arg main_camera)">
@@ -16,254 +17,15 @@
     <xacro:distance_sensor parent="base_link" x="0.0" y="0.0" z="-0.04" roll="0" pitch="${M_PI / 2}" yaw="0"/>
   </xacro:if>
-  <!-- Add LED strip model TODO: redo -->
-  <joint name="led_strip_joint" type="fixed">
-    <origin xyz="0 0 0"
-            rpy="0 0 0"/>
-    <parent link="base_link"/>
-    <child link="led_link"/>
-  </joint>
-  <!-- TODO: remove hardcode -->
-  <link name="led_link">
-    <visual name="led_0_visual">
-      <origin rpy="0  0  0" xyz="0    0.08  0"/>
-      <geometry>
-        <sphere radius="0.005"/>
-      </geometry>
-    </visual>
-    <visual name="led_1_visual">
-      <origin rpy="0  0  0" xyz="0.01251  0.07901  0"/>
-      <geometry>
-        <sphere radius="0.005"/>
-      </geometry>
-    </visual>
-    <visual name="led_2_visual">
-      <origin rpy="0  0  0" xyz="0.02472  0.07608  0"/>
-      <geometry>
-        <sphere radius="0.005"/>
-      </geometry>
-    </visual>
-    <visual name="led_3_visual">
-      <origin rpy="0  0  0" xyz="0.03631  0.07128  0"/>
-      <geometry>
-        <sphere radius="0.005"/>
-      </geometry>
-    </visual>
-    <visual name="led_4_visual">
-      <origin rpy="0  0  0" xyz="0.04702  0.06472  0"/>
-      <geometry>
-        <sphere radius="0.005"/>
-      </geometry>
-    </visual>
-    <visual name="led_5_visual">
-      <origin rpy="0  0  0" xyz="0.05656  0.05656  0"/>
-      <geometry>
-        <sphere radius="0.005"/>
-      </geometry>
-    </visual>
-    <visual name="led_6_visual">
-      <origin rpy="0  0  0" xyz="0.06472  0.04702  0"/>
-      <geometry>
-        <sphere radius="0.005"/>
-      </geometry>
-    </visual>
-    <visual name="led_7_visual">
-      <origin rpy="0  0  0" xyz="0.07128  0.03631  0"/>
-      <geometry>
-        <sphere radius="0.005"/>
-      </geometry>
-    </visual>
-    <visual name="led_8_visual">
-      <origin rpy="0  0  0" xyz="0.07608  0.02472  0"/>
-      <geometry>
-        <sphere radius="0.005"/>
-      </geometry>
-    </visual>
-    <visual name="led_9_visual">
-      <origin rpy="0  0  0" xyz="0.07901  0.01251  0"/>
-      <geometry>
-        <sphere radius="0.005"/>
-      </geometry>
-    </visual>
-    <visual name="led_10_visual">
-      <origin rpy="0  0  0" xyz="0.08  0    0"/>
-      <geometry>
-        <sphere radius="0.005"/>
-      </geometry>
-    </visual>
-    <visual name="led_11_visual">
-      <origin rpy="0  0  0" xyz="0.07901 -0.01251  0"/>
-      <geometry>
-        <sphere radius="0.005"/>
-      </geometry>
-    </visual>
-    <visual name="led_12_visual">
-      <origin rpy="0  0  0" xyz="0.07608 -0.02472  0"/>
-      <geometry>
-        <sphere radius="0.005"/>
-      </geometry>
-    </visual>
-    <visual name="led_13_visual">
-      <origin rpy="0  0  0" xyz="0.07128 -0.03631  0"/>
-      <geometry>
-        <sphere radius="0.005"/>
-      </geometry>
-    </visual>
-    <visual name="led_14_visual">
-      <origin rpy="0  0  0" xyz="0.06472 -0.04702  0"/>
-      <geometry>
-        <sphere radius="0.005"/>
-      </geometry>
-    </visual>
-    <visual name="led_15_visual">
-      <origin rpy="0  0  0" xyz="0.05656 -0.05656  0"/>
-      <geometry>
-        <sphere radius="0.005"/>
-      </geometry>
-    </visual>
-    <visual name="led_16_visual">
-      <origin rpy="0  0  0" xyz="0.04702 -0.06472  0"/>
-      <geometry>
-        <sphere radius="0.005"/>
-      </geometry>
-    </visual>
-    <visual name="led_17_visual">
-      <origin rpy="0  0  0" xyz="0.03631 -0.07128  0"/>
-      <geometry>
-        <sphere radius="0.005"/>
-      </geometry>
-    </visual>
-    <visual name="led_18_visual">
-      <origin rpy="0  0  0" xyz="0.02472 -0.07608  0"/>
-      <geometry>
-        <sphere radius="0.005"/>
-      </geometry>
-    </visual>
-    <visual name="led_19_visual">
-      <origin rpy="0  0  0" xyz="0.01251 -0.07901  0"/>
-      <geometry>
-        <sphere radius="0.005"/>
-      </geometry>
-    </visual>
-    <visual name="led_20_visual">
-      <origin rpy="0  0  0" xyz="0   -0.08  0"/>
-      <geometry>
-        <sphere radius="0.005"/>
-      </geometry>
-    </visual>
-    <visual name="led_21_visual">
-      <origin rpy="0  0  0" xyz="-0.01251 -0.07901  0"/>
-      <geometry>
-        <sphere radius="0.005"/>
-      </geometry>
-    </visual>
-    <visual name="led_22_visual">
-      <origin rpy="0  0  0" xyz="-0.02472 -0.07608  0"/>
-      <geometry>
-        <sphere radius="0.005"/>
-      </geometry>
-    </visual>
-    <visual name="led_23_visual">
-      <origin rpy="0  0  0" xyz="-0.03631 -0.07128  0"/>
-      <geometry>
-        <sphere radius="0.005"/>
-      </geometry>
-    </visual>
-    <visual name="led_24_visual">
-      <origin rpy="0  0  0" xyz="-0.04702 -0.06472  0"/>
-      <geometry>
-        <sphere radius="0.005"/>
-      </geometry>
-    </visual>
-    <visual name="led_25_visual">
-      <origin rpy="0  0  0" xyz="-0.05656 -0.05656  0"/>
-      <geometry>
-        <sphere radius="0.005"/>
-      </geometry>
-    </visual>
-    <visual name="led_26_visual">
-      <origin rpy="0  0  0" xyz="-0.06472 -0.04702  0"/>
-      <geometry>
-        <sphere radius="0.005"/>
-      </geometry>
-    </visual>
-    <visual name="led_27_visual">
-      <origin rpy="0  0  0" xyz="-0.07128 -0.03631  0"/>
-      <geometry>
-        <sphere radius="0.005"/>
-      </geometry>
-    </visual>
-    <visual name="led_28_visual">
-      <origin rpy="0  0  0" xyz="-0.07608 -0.02472  0"/>
-      <geometry>
-        <sphere radius="0.005"/>
-      </geometry>
-    </visual>
-    <visual name="led_29_visual">
-      <origin rpy="0  0  0" xyz="-0.07901 -0.01251  0"/>
-      <geometry>
-        <sphere radius="0.005"/>
-      </geometry>
-    </visual>
-    <visual name="led_30_visual">
-      <origin rpy="0  0  0" xyz="-0.08  0    0"/>
-      <geometry>
-        <sphere radius="0.005"/>
-      </geometry>
-    </visual>
-    <visual name="led_31_visual">
-      <origin rpy="0  0  0" xyz="-0.07901  0.01251  0"/>
-      <geometry>
-        <sphere radius="0.005"/>
-      </geometry>
-    </visual>
-    <visual name="led_32_visual">
-      <origin rpy="0  0  0" xyz="-0.07608  0.02472  0"/>
-      <geometry>
-        <sphere radius="0.005"/>
-      </geometry>
-    </visual>
-    <visual name="led_33_visual">
-      <origin rpy="0  0  0" xyz="-0.07128  0.03631  0"/>
-      <geometry>
-        <sphere radius="0.005"/>
-      </geometry>
-    </visual>
-    <visual name="led_34_visual">
-      <origin rpy="0  0  0" xyz="-0.06472  0.04702  0"/>
-      <geometry>
-        <sphere radius="0.005"/>
-      </geometry>
-    </visual>
-    <visual name="led_35_visual">
-      <origin rpy="0  0  0" xyz="-0.05656  0.05656  0"/>
-      <geometry>
-        <sphere radius="0.005"/>
-      </geometry>
-    </visual>
-    <visual name="led_36_visual">
-      <origin rpy="0  0  0" xyz="-0.04702  0.06472  0"/>
-      <geometry>
-        <sphere radius="0.005"/>
-      </geometry>
-    </visual>
-    <visual name="led_37_visual">
-      <origin rpy="0  0  0" xyz="-0.03631  0.07128  0"/>
-      <geometry>
-        <sphere radius="0.005"/>
-      </geometry>
-    </visual>
-    <visual name="led_38_visual">
-      <origin rpy="0  0  0" xyz="-0.02472  0.07608  0"/>
-      <geometry>
-        <sphere radius="0.005"/>
-      </geometry>
-    </visual>
-    <visual name="led_39_visual">
-      <origin rpy="0  0  0" xyz="-0.01251  0.07901  0"/>
-      <geometry>
-        <sphere radius="0.005"/>
-      </geometry>
-    </visual>
-  </link>
+  <!-- Instantiate LED strip -->
+  <xacro:if value="$(arg led)">
+    <xacro:led_strip
+      name="led"
+      parent="base_link"
+      radius="0.08"
+      bulb_radius="0.006"
+      led_count="58"
+      use_plugin="true"
+      z="-0.002"/>
+  </xacro:if>
   <xacro:if value="$(arg gps)">
     <!-- Instantiate gps plugin. -->
@@ -271,6 +33,5 @@
       namespace="${namespace}"
       gps_noise="true"
-      >
-    </xacro:gps_plugin_macro>
+      />
   </xacro:if>
 </robot>

Commit message: clover_description: Add calculated inertial parameters

File: clover_description/urdf/clover/clover4.xacro (robot description, xacro)
@@ -6,4 +6,5 @@
   <xacro:arg name="gps" default="true"/>
   <xacro:arg name="maintain_camera_rate" default="false"/>
+  <xacro:arg name="use_clover_physics" default="false"/>
   <xacro:include filename="$(find clover_description)/urdf/clover/clover4_base.xacro" />
   <xacro:include filename="$(find clover_description)/urdf/sensors/rpi_cam.urdf.xacro"/>

File: clover_description/urdf/clover/clover4_physics.xacro (robot description, xacro)
@@ -8,5 +8,10 @@
   <xacro:property name="namespace" value="" />
   <xacro:property name="rotor_velocity_slowdown_sim" value="10" />
-  <xacro:property name="mass" value="1.5" /> <!-- [kg] -->
+  <xacro:if value="$(arg use_clover_physics)">
+    <xacro:property name="mass" value="0.7" /> <!-- [kg] -->
+  </xacro:if>
+  <xacro:unless value="$(arg use_clover_physics)">
+    <xacro:property name="mass" value="1.5" /> <!-- [kg] -->
+  </xacro:unless>
   <xacro:property name="body_width" value="0.35" /> <!-- [m] -->
   <xacro:property name="body_height" value="0.124" /> <!-- [m] -->
@@ -30,19 +35,46 @@
   <xacro:property name="color" value="$(arg visual_material)" />
   <!-- Property Blocks -->
-  <xacro:property name="body_inertia">
-    <inertia
-    ixx="${1/12 * mass * (body_height * body_height + body_width * body_width)}"
-    iyy="${1/12 * mass * (body_height * body_height + body_width * body_width)}"
-    izz="${1/12 * mass * (body_width * body_width + body_width * body_width)}"
-    ixy="0.0" ixz="0.0" iyz="0.0" /> <!-- [kg.m^2] [kg.m^2] [kg.m^2] [kg.m^2] [kg.m^2] [kg.m^2] -->
-  </xacro:property>
-  <!-- inertia of a single rotor, assuming it is a cuboid. Height=3mm, width=15mm -->
-  <xacro:property name="rotor_inertia">
-    <inertia
-    ixx="${1/12 * mass_rotor * (0.015 * 0.015 + 0.003 * 0.003) * rotor_velocity_slowdown_sim}"
-    iyy="${1/12 * mass_rotor * (4 * radius_rotor * radius_rotor + 0.003 * 0.003) * rotor_velocity_slowdown_sim}"
-    izz="${1/12 * mass_rotor * (4 * radius_rotor * radius_rotor + 0.015 * 0.015) * rotor_velocity_slowdown_sim}"
-    ixy="0.0" ixz="0.0"  iyz="0.0" /> <!-- [kg.m^2] [kg.m^2] [kg.m^2] [kg.m^2] [kg.m^2] [kg.m^2] -->
-  </xacro:property>
+  <!-- Clover body inertia -->
+  <!-- Values from CAD program -->
+  <xacro:if value="$(arg use_clover_physics)">
+    <xacro:property name="body_inertia">
+      <inertia
+      ixx="0.0347563"
+      iyy="0.0458929"
+      izz="0.0977"
+      ixy="0.0" ixz="0.0" iyz="0.0" /> <!-- [kg.m^2] [kg.m^2] [kg.m^2] [kg.m^2] [kg.m^2] [kg.m^2] -->
+    </xacro:property>
+  </xacro:if>
+  <!-- Box-like inertia -->
+  <xacro:unless value="$(arg use_clover_physics)">
+    <xacro:property name="body_inertia">
+      <inertia
+      ixx="${1/12 * mass * (body_height * body_height + body_width * body_width)}"
+      iyy="${1/12 * mass * (body_height * body_height + body_width * body_width)}"
+      izz="${1/12 * mass * (body_width * body_width + body_width * body_width)}"
+      ixy="0.0" ixz="0.0" iyz="0.0" /> <!-- [kg.m^2] [kg.m^2] [kg.m^2] [kg.m^2] [kg.m^2] [kg.m^2] -->
+    </xacro:property>
+  </xacro:unless>
+  <!-- inertia of a single rotor -->
+  <!-- Values from CAD program -->
+  <xacro:if value="$(arg use_clover_physics)">
+    <xacro:property name="rotor_inertia">
+      <inertia
+      ixx="${1.375 * 0.001 * 0.001 * rotor_velocity_slowdown_sim}"
+      iyy="${2.153 * 0.001 * 0.001 * rotor_velocity_slowdown_sim}"
+      izz="${1.375 * 0.001 * 0.001 * rotor_velocity_slowdown_sim}"
+      ixy="0.0" ixz="0.0"  iyz="0.0" /> <!-- [kg.m^2] [kg.m^2] [kg.m^2] [kg.m^2] [kg.m^2] [kg.m^2] -->
+    </xacro:property>
+  </xacro:if>
+  <!-- Values for a cuboid (cuboid. Height=3mm, width=15mm) -->
+  <xacro:unless value="$(arg use_clover_physics)">
+    <xacro:property name="rotor_inertia">
+      <inertia
+      ixx="${1/12 * mass_rotor * (0.015 * 0.015 + 0.003 * 0.003) * rotor_velocity_slowdown_sim}"
+      iyy="${1/12 * mass_rotor * (4 * radius_rotor * radius_rotor + 0.003 * 0.003) * rotor_velocity_slowdown_sim}"
+      izz="${1/12 * mass_rotor * (4 * radius_rotor * radius_rotor + 0.015 * 0.015) * rotor_velocity_slowdown_sim}"
+      ixy="0.0" ixz="0.0"  iyz="0.0" /> <!-- [kg.m^2] [kg.m^2] [kg.m^2] [kg.m^2] [kg.m^2] [kg.m^2] -->
+    </xacro:property>
+  </xacro:unless>
   <!-- Included URDF Files -->
   <xacro:include filename="$(find clover_description)/urdf/clover/clover4_macros.xacro" />
