Commit message: clover_description: simplify URDF and copy Gazebo plugins from current PX4’s Iris

File: clover_description/urdf/clover/clover4.xacro (robot description, xacro)
@@ -1,4 +1,4 @@
 <?xml version="1.0"?>
-<robot name="clover_camera" xmlns:xacro="http://ros.org/wiki/xacro">
+<robot name="clover" xmlns:xacro="http://ros.org/wiki/xacro">
   <xacro:arg name="main_camera" default="true"/>
   <xacro:arg name="rangefinder" default="true"/>

File: clover_description/urdf/clover/clover4_base.xacro (robot description, xacro)
@@ -1,32 +1,7 @@
 <?xml version="1.0"?>
 <robot name="clover" xmlns:xacro="http://ros.org/wiki/xacro">
-  <!-- Properties that can be assigned at build time as arguments.
-  Is there a reason not to make all properties arguments?
-  -->
-  <xacro:arg name='name' default='iris' />
-  <xacro:arg name='mavlink_addr' default='INADDR_ANY' />
-  <xacro:arg name='mavlink_udp_port' default='14560' />
-  <xacro:arg name='mavlink_tcp_port' default='4560' />
-  <xacro:arg name='serial_enabled' default='false' />
-  <xacro:arg name='serial_device' default='/dev/ttyACM0' />
-  <xacro:arg name='baudrate' default='921600' />
-  <xacro:arg name='qgc_addr' default='INADDR_ANY' />
-  <xacro:arg name='qgc_udp_port' default='14550' />
-  <xacro:arg name='sdk_addr' default='INADDR_ANY' />
-  <xacro:arg name='sdk_udp_port' default='14540' />
-  <xacro:arg name='hil_mode' default='false' />
-  <xacro:arg name='hil_state_level' default='false' />
-  <xacro:arg name='send_vision_estimation' default='false' />
-  <xacro:arg name='send_odometry' default='false' />
-  <xacro:arg name='enable_lockstep' default='true' />
-  <xacro:arg name='use_tcp' default='true' />
-  <xacro:arg name='vehicle_is_tailsitter' default='false' />
-  <xacro:arg name='visual_material' default='DarkGrey' />
-  <xacro:arg name='enable_mavlink_interface' default='true' />
   <xacro:arg name='enable_wind' default='false' />
-  <!-- The following causes segfault with multiple vehicles if defaults to true!!! -->
-  <xacro:arg name='enable_ground_truth' default='false' />
   <xacro:arg name='enable_logging' default='false' />
-  <xacro:arg name='log_file' default='iris' />
+  <xacro:arg name='log_file' default='clover' />
   <!-- macros for gazebo plugins, sensors -->
   <xacro:include filename="../component_snippets.urdf.xacro" />
@@ -45,119 +20,6 @@
         />
   </xacro:if>
-  <!-- Instantiate magnetometer plugin. -->
-  <xacro:magnetometer_plugin_macro
-    namespace="${namespace}"
-    pub_rate="20"
-    noise_density="0.0004"
-    random_walk="0.0000064"
-    bias_correlation_time="600"
-    mag_topic="/mag"
-    >
-  </xacro:magnetometer_plugin_macro>
-  <!-- Instantiate barometer plugin. -->
-  <xacro:barometer_plugin_macro
-    namespace="${namespace}"
-    pub_rate="10"
-    baro_topic="/baro"
-    >
-  </xacro:barometer_plugin_macro>
-  <xacro:if value="$(arg enable_mavlink_interface)">
-  <!-- Instantiate mavlink telemetry interface. -->
-  <xacro:mavlink_interface_macro
-    namespace="${namespace}"
-    imu_sub_topic="/imu"
-    gps_sub_topic="/gps"
-    mag_sub_topic="/mag"
-    baro_sub_topic="/baro"
-    mavlink_addr="$(arg mavlink_addr)"
-    mavlink_udp_port="$(arg mavlink_udp_port)"
-    mavlink_tcp_port="$(arg mavlink_tcp_port)"
-    serial_enabled="$(arg serial_enabled)"
-    serial_device="$(arg serial_device)"
-    baudrate="$(arg baudrate)"
-    qgc_addr="$(arg qgc_addr)"
-    qgc_udp_port="$(arg qgc_udp_port)"
-    sdk_addr="$(arg sdk_addr)"
-    sdk_udp_port="$(arg sdk_udp_port)"
-    hil_mode="$(arg hil_mode)"
-    hil_state_level="$(arg hil_state_level)"
-    vehicle_is_tailsitter="$(arg vehicle_is_tailsitter)"
-    send_vision_estimation="$(arg send_vision_estimation)"
-    send_odometry="$(arg send_odometry)"
-    enable_lockstep="$(arg enable_lockstep)"
-    use_tcp="$(arg use_tcp)"
-    >
-  </xacro:mavlink_interface_macro>
-  </xacro:if>
-  <!-- Mount an ADIS16448 IMU. -->
-  <xacro:imu_plugin_macro
-    namespace="${namespace}"
-    imu_suffix=""
-    parent_link="base_link"
-    imu_topic="/imu"
-    mass_imu_sensor="0.015"
-    gyroscope_noise_density="0.0003394"
-    gyroscopoe_random_walk="0.000038785"
-    gyroscope_bias_correlation_time="1000.0"
-    gyroscope_turn_on_bias_sigma="0.0087"
-    accelerometer_noise_density="0.004"
-    accelerometer_random_walk="0.006"
-    accelerometer_bias_correlation_time="300.0"
-    accelerometer_turn_on_bias_sigma="0.1960"
-  >
-    <inertia ixx="0.00001" ixy="0.0" ixz="0.0" iyy="0.00001" iyz="0.0" izz="0.00001" />
-    <origin xyz="0 0 0" rpy="0 0 0" />
-  </xacro:imu_plugin_macro>
-  <xacro:if value="$(arg enable_ground_truth)">
-    <!-- Mount an IMU providing ground truth. -->
-    <xacro:imu_plugin_macro
-      namespace="${namespace}"
-      imu_suffix="gt"
-      parent_link="base_link"
-      imu_topic="ground_truth/imu"
-      mass_imu_sensor="0.00001"
-      gyroscope_noise_density="0.0"
-      gyroscopoe_random_walk="0.0"
-      gyroscope_bias_correlation_time="1000.0"
-      gyroscope_turn_on_bias_sigma="0.0"
-      accelerometer_noise_density="0.0"
-      accelerometer_random_walk="0.0"
-      accelerometer_bias_correlation_time="300.0"
-      accelerometer_turn_on_bias_sigma="0.0"
-    >
-      <inertia ixx="0.00001" ixy="0.0" ixz="0.0" iyy="0.00001" iyz="0.0" izz="0.00001" />
-      <origin xyz="0 0 0" rpy="0 0 0" />
-    </xacro:imu_plugin_macro>
-    <!-- Mount a generic odometry sensor providing ground truth. -->
-    <xacro:odometry_plugin_macro
-      namespace="${namespace}/ground_truth"
-      odometry_sensor_suffix="gt"
-      parent_link="base_link"
-      pose_topic="pose"
-      pose_with_covariance_topic="pose_with_covariance"
-      position_topic="position"
-      transform_topic="transform"
-      odometry_topic="odometry"
-      parent_frame_id="world"
-      mass_odometry_sensor="0.00001"
-      measurement_divisor="1"
-      measurement_delay="0"
-      unknown_delay="0.0"
-      noise_normal_position="0 0 0"
-      noise_normal_quaternion="0 0 0"
-      noise_normal_linear_velocity="0 0 0"
-      noise_normal_angular_velocity="0 0 0"
-      noise_uniform_position="0 0 0"
-      noise_uniform_quaternion="0 0 0"
-      noise_uniform_linear_velocity="0 0 0"
-      noise_uniform_angular_velocity="0 0 0"
-      enable_odometry_map="false"
-      odometry_map=""
-      image_scale=""
-    >
-      <inertia ixx="0.00001" ixy="0.0" ixz="0.0" iyy="0.00001" iyz="0.0" izz="0.00001" /> <!-- [kg.m^2] [kg.m^2] [kg.m^2] [kg.m^2] [kg.m^2] [kg.m^2] -->
-      <origin xyz="0.0 0.0 0.0" rpy="0.0 0.0 0.0" />
-    </xacro:odometry_plugin_macro>
-  </xacro:if>
+  <!-- Gazebo plugins -->
+  <xacro:include filename="$(find clover_description)/urdf/clover/clover4_gazebo.xacro" />
   <xacro:if value="$(arg enable_logging)">
     <!-- Instantiate a logger -->

File: clover_description/urdf/clover/clover4_physics.xacro (robot description, xacro)
@@ -4,5 +4,5 @@
      This is subject to change as correct values are calculated.
 -->
-<robot name="iris" xmlns:xacro="http://ros.org/wiki/xacro">
+<robot name="clover" xmlns:xacro="http://ros.org/wiki/xacro">
   <!-- Properties -->
   <xacro:property name="namespace" value="" />

Commit message: clover_description: fix gps sensor

File: clover_description/urdf/clover/clover4.xacro (robot description, xacro)
@@ -31,9 +31,15 @@
   </xacro:if>
   <xacro:if value="$(arg gps)">
-    <!-- Instantiate gps plugin. -->
-    <xacro:gps_plugin_macro
-      namespace="${namespace}"
-      gps_noise="true"
-      />
+    <gazebo>
+      <include>
+        <uri>model://gps</uri>
+        <pose>0.1 0 0 0 0 0</pose>
+        <name>gps0</name>
+      </include>
+      <joint name='gps0_joint' type='fixed'>
+        <child>gps0::link</child>
+        <parent>base_link</parent>
+      </joint>
+    </gazebo>
   </xacro:if>
 </robot>

Commit message: changing size of led_ring

File: clover_description/urdf/clover/clover4.xacro (robot description, xacro)
@@ -14,5 +14,5 @@
   <!-- Create camera plugin -->
   <xacro:if value="$(arg main_camera)">
-    <xacro:rpi_cam name="main_camera" parent="base_link" x="0.055" y="0.0" z="-0.03" roll="0" pitch="${pi / 2}" yaw="0" width="320" height="240" rate="40" do_throttling="$(arg maintain_camera_rate)"/>
+    <xacro:rpi_cam name="main_camera" parent="base_link" x="0.055" y="0.0" z="-0.03" roll="0" pitch="${pi/2}" yaw="0" width="320" height="240" rate="40" do_throttling="$(arg maintain_camera_rate)"/>
   </xacro:if>
   <!-- Instantiate LED strip -->
@@ -21,7 +21,7 @@
       name="led"
       parent="base_link"
-      radius="0.08"
-      bulb_radius="0.006"
-      led_count="58"
+      radius="0.1"
+      bulb_radius="0.01"
+      led_count="72"
       use_plugin="true"
       z="-0.002"/>

File: clover_description/urdf/leds/led_strip.xacro (robot description, xacro)
@@ -28,5 +28,5 @@
                             rpy="0 0 ${2 * pi * link_i / links_total}"/>
                     <geometry>
-                        <box size="${bulb_radius} ${bulb_radius} ${bulb_radius}"/>
+                        <box size="${bulb_radius} ${bulb_radius} ${2 * bulb_radius}"/>
                     </geometry>
                 </visual>
