Commit message: Minor fixes

File: clover_description/urdf/leds/led_strip.xacro (robot description, xacro)
@@ -28,5 +28,5 @@
                             rpy="0 0 ${2 * pi * link_i / links_total}"/>
                     <geometry>
-                        <box size="${bulb_radius} ${bulb_radius} ${2 * bulb_radius}"/>
+                        <box size="${bulb_radius} ${bulb_radius} ${bulb_radius}"/>
                     </geometry>
                 </visual>
